File: KiCad Project Files/UWU PDB.kicad_pcb (KiCad board)
At the start: 4 copper layers, 96.5 x 92.2 mm, 77 parts, among them J1 XT90, J10 XT60 ESC, J11 PWM ESC, J12 PWM ESC, J13 PWM ESC, J14 PWM ESC, J15 PWM ESC, J16 PWM ESC, J17 PWM ESC, J18 PWM ESC, J19 XT90, J2 Conn_02x08_Odd_Even, J3 XT60 ESC, J4 XT60 ESC, J5 XT60 ESC, J6 XT60 ESC, J7 XT60 ESC, J8 XT60 ESC, J9 XT60 ESC

Commit message: v1.1 PCB
Parts:
- moved REF** 0.97 mm to (175.3, 111.8)
- moved REF** 0.20 mm to (84.2, 111.8)
Routing:
- net /VBAT+: vias 60 -> 58
